File: Docs/Documents & Advanced/PCB/V3.3/einkPDA_screen/einkPDA_screen.kicad_pcb (KiCad board)
At the start: 2 copper layers, 95 x 54 mm, 29 parts, among them J3 CapacitiveTouch, J4 Conn_01x12_Pin, Q1 Si1308EDL, U1 MPR121QR2

Commit message: PCB V3.3
Parts:
- removed R4: 1R, Resistor_SMD:R_0603_1608Metric
- R1: value 1R -> 0.47R
Routing:
- net RESE: track 51.8 -> 49.6 mm
- net GND: track 6.65 -> 6.48 mm, vias 166 -> 168
