File: Docs/Documents & Advanced/PCB/V3.3/einkPDA_screen/einkPDA_screen.kicad_sch (KiCad schematic)
At the start: 28 parts, among them J3 CapacitiveTouch, J4 Conn_01x12_Pin, Q1 Si1308EDL, U1 MPR121QR2

Commit message: PCB V3.3
Parts:
- removed R4: 1R, Resistor_SMD:R_0603_1608Metric, symbol Device:R
- C1, C10, C3, C4, C5, C6, C7, C8, C9: MPN CL05A105KA5NQNC -> C52923
- C11: MPN CL21A475KAQNNNE -> C1779
- C12, C2: MPN CL05A475MP5NRNC -> C23733
- C13, C14: MPN CL05B104KO5NNNC -> C1525
- D1, D2, D3: MPN MBR0530 -> C77336
- J2: MPN AFE03-S25FMA-1H -> C262544
- J4: MPN AFC01-S12FCA-00 -> C262661
- L1: MPN SWPA5020S100MT -> C52281
- Q1: MPN Si1308EDL -> C7603347
- R1: value 1R -> 0.47R; MPN 0603WAF100KT5E -> C3013349
- R2: MPN 0805W8F1002T5E -> C17414
- R3: MPN 0603WAF7502T5E -> C23242
- RN1: MPN 4D03WGJ0103T5E -> C29718
- U1: MPN MPR121QR2 -> C91322
Changed lines of the file:
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@@
 	)
 	(junction
-		(at 48.26 82.55)
-		(diameter 0)
-		(color 0 0 0 0)
-	)
-	(junction
 		(at 73.66 48.26)
 		(diameter 0)
@@
 	)
 	(junction
-		(at 48.26 74.93)
-		(diameter 0)
-		(color 0 0 0 0)
-	)
-	(junction
 		(at 26.67 48.26)
 		(diameter 0)
@@
 	(wire
 		(pts
-			(xy 48.26 82.55) (xy 55.88 82.55)
-		)
-		(stroke
-			(width 0)
-			(type default)
-		)
-	)
-	(wire
-		(pts
 			(xy 124.46 54.61) (xy 130.81 54.61)
 		)
@@
 	(wire
 		(pts
-			(xy 55.88 74.93) (xy 48.26 74.93)
-		)
-		(stroke
-			(width 0)
-			(type default)
-		)
-	)
-	(wire
-		(pts
 			(xy 81.28 120.65) (xy 96.52 120.65)
 		)
@@
 			)
 		)
-		(property "MPN" "MPR121QR2"
+		(property "MPN" "C91322"
 			(at 109.22 115.57 0)
 			(effects
@@
 			)
 		)
-		(property "MPN" "CL05A105KA5NQNC"
+		(property "MPN" "C52923"
 			(at 166.37 52.07 0)
 			(effects
@@
 			)
 		)
-		(property "MPN" "AFE03-S25FMA-1H"
+		(property "MPN" "C262544"
 			(at 135.89 29.21 0)
 			(effects
@@
 			)
 		)
-		(property "MPN" "CL05A105KA5NQNC"
+		(property "MPN" "C52923"
 			(at 172.72 66.04 0)
 			(effects
@@
 			)
 		)
-		(property "MPN" "CL21A475KAQNNNE"
+		(property "MPN" "C1779"
 			(at 48.26 39.37 0)
 			(effects
@@
 			)
 		)
-		(property "MPN" "CL05A105KA5NQNC"
+		(property "MPN" "C52923"
 			(at 73.66 52.07 0)
 			(effects
@@
 			)
 		)
-		(property "MPN" "CL05B104KO5NNNC"
+		(property "MPN" "C1525"
 			(at 96.52 91.44 0)
 			(effects
@@
 			)
 		)
-		(property "MPN" "AFC01-S12FCA-00"
+		(property "MPN" "C262661"
 			(at 209.55 109.22 0)
 			(effects
@@
 			)
 		)
-		(property "MPN" "MBR0530"
+		(property "MPN" "C77336"
 			(at 64.77 48.26 0)
 			(effects
@@
 			)
 		)
-		(property "MPN" "CL05A105KA5NQNC"
+		(property "MPN" "C52923"
 			(at 172.72 34.29 0)
 			(effects
@@
 			)
 		)
-		(property "MPN" "Si1308EDL"
+		(property "MPN" "C7603347"
 			(at 45.72 60.96 0)
 			(effects
@@
 			)
 		)
-		(property "MPN" "CL05A475MP5NRNC"
+		(property "MPN" "C23733"
 			(at 116.84 36.83 0)
 			(effects
@@
 			)
 		)
-		(property "MPN" "MBR0530"
+		(property "MPN" "C77336"
 			(at 64.77 35.56 0)
 			(effects
@@
 			)
 		)
-		(property "Value" "1R"
+		(property "Value" "0.47R"
 			(at 50.8 80.0099 0)
 			(effects
@@
 			)
 		)
-		(property "MPN" "0603WAF100KT5E"
+		(property "MPN" "C3013349"
 			(at 48.26 78.74 0)
 			(effects
@@
 			)
 		)
-		(property "MPN" "MBR0530"
+		(property "MPN" "C77336"
 			(at 64.77 24.13 0)
 			(effects
@@
 			)
 		)
-		(property "MPN" "0603WAF7502T5E"
+		(property "MPN" "C23242"
 			(at 81.28 127 0)
 			(effects
@@
 			)
 		)
-		(property "MPN" "CL05A105KA5NQNC"
+		(property "MPN" "C52923"
 			(at 120.65 54.61 0)
 			(effects
@@
 	)
 	(symbol
-		(lib_id "Device:R")
-		(at 55.88 78.74 0)
-		(unit 1)
-		(exclude_from_sim no)
-		(in_bom yes)
-		(on_board yes)
-		(dnp no)
-		(fields_autoplaced yes)
-		(property "Reference" "R4"
-			(at 58.42 77.4699 0)
-			(effects
-				(font
-					(size 1.27 1.27)
-				)
-				(justify left)
-			)
-		)
-		(property "Value" "1R"
-			(at 58.42 80.0099 0)
-			(effects
-				(font
-					(size 1.27 1.27)
-				)
-				(justify left)
-			)
-		)
-		(property "Footprint" "Resistor_SMD:R_0603_1608Metric"
-			(at 54.102 78.74 90)
-			(effects
-				(font
-					(size 1.27 1.27)
-				)
-				(hide yes)
-			)
-		)
-		(property "Datasheet" "~"
-			(at 55.88 78.74 0)
-			(effects
-				(font
-					(size 1.27 1.27)
-				)
-				(hide yes)
-			)
-		)
-		(property "Description" "Resistor"
-			(at 55.88 78.74 0)
-			(effects
-				(font
-					(size 1.27 1.27)
-				)
-				(hide yes)
-			)
-		)
-		(property "Height" ""
-			(at 55.88 78.74 0)
-			(effects
-				(font
-					(size 1.27 1.27)
-				)
-				(hide yes)
-			)
-		)
-		(property "Manufacturer_Name" ""
-			(at 55.88 78.74 0)
-			(effects
-				(font
-					(size 1.27 1.27)
-				)
-				(hide yes)
-			)
-		)
-		(property "Mouser Part Number" ""
-			(at 55.88 78.74 0)
-			(effects
-				(font
-					(size 1.27 1.27)
-				)
-				(hide yes)
-			)
-		)
-		(property "Mouser Price/Stock" ""
-			(at 55.88 78.74 0)
-			(effects
-				(font
-					(size 1.27 1.27)
-				)
-				(hide yes)
-			)
-		)
-		(property "MPN" "0603WAF100KT5E"
-			(at 55.88 78.74 0)
-			(effects
-				(font
-					(size 1.27 1.27)
-				)
-				(hide yes)
-			)
-		)
-		(pin "1"
-		)
-		(pin "2"
-		)
-		(instances
-			(project "einkPDA_screen"
-				(path "/8cfe7814-b2da-47eb-a463-3cc98c19cb36"
-					(reference "R4")
-					(unit 1)
-				)
-			)
-		)
-	)
-	(symbol
 		(lib_id "Device:C")
 		(at 90.17 129.54 0)
@@
 			)
 		)
-		(property "MPN" "CL05B104KO5NNNC"
+		(property "MPN" "C1525"
 			(at 90.17 129.54 0)
 			(effects
@@
 			)
 		)
-		(property "MPN" "0805W8F1002T5E"
+		(property "MPN" "C17414"
 			(at 38.1 78.74 0)
 			(effects
@@
 			)
 		)
-		(property "MPN" "4D03WGJ0103T5E"
+		(property "MPN" "C29718"
 			(at 78.74 110.49 0)
 			(effects
@@
 			)
 		)
-		(property "MPN" "CL05A105KA5NQNC"
+		(property "MPN" "C52923"
 			(at 162.56 57.15 0)
 			(effects
@@
 			)
 		)
-		(property "MPN" "CL05A105KA5NQNC"
+		(property "MPN" "C52923"
 			(at 116.84 59.69 0)
 			(effects
@@
 			)
 		)
-		(property "MPN" "CL05A105KA5NQNC"
+		(property "MPN" "C52923"
 			(at 172.72 54.61 0)
 			(effects
@@
 			)
 		)
-		(property "MPN" "CL05A105KA5NQNC"
+		(property "MPN" "C52923"
 			(at 116.84 49.53 0)
 			(effects
@@
 			)
 		)
-		(property "MPN" "CL05A475MP5NRNC"
+		(property "MPN" "C23733"
 			(at 26.67 52.07 0)
 			(effects
@@
 			)
 		)
-		(property "MPN" "SWPA5020S100MT"
+		(property "MPN" "C52281"
 			(at 38.1 48.26 0)
 			(effects
