File: Docs/Documents & Advanced/PCB/V3.3/einkPDA_keyboard/einkPDA_keyboard.kicad_sch (KiCad schematic)
At the start: 140 parts, among them J1 USB_C_Receptacle_USB2.0_16P, J2 Conn_01x12_Pin, J3 Conn_01x26_Pin, J4 Micro_SD_Card, J5 Conn_01x12_Pin, Q1 MMBT3904, SW36 YTS-C017-2B, SW4 SW_DIP_x02, SW41 YTS-C017-2B, U1 ESP32-S3-WROOM-1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

Commit message: PCB V3.3
Changed lines of the file:
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@@
 	(text "Sleep Load Switch"
 		(exclude_from_sim no)
-		(at 157.734 259.08 0)
+		(at 157.734 259.842 0)
 		(effects
 			(font

Commit message: PCB updates
Parts:
- L3: LCSC Part # C19734 -> C167747
- SW36, SW41: LCSC Part # (none) -> C2910872
- U1: LCSC Part # C2913202 -> C2913205
- U8: LCSC Part # (none) -> C2681320
Changed lines of the file:
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@@
 			)
 		)
+		(property "LCSC Part #" "C2910872"
+			(at 30.48 133.35 0)
+			(effects
+				(font
+					(size 1.27 1.27)
+				)
+				(hide yes)
+			)
+		)
 		(pin "2"
 		)
@@
 			)
 		)
+		(property "LCSC Part #" "C2910872"
+			(at 34.29 114.3 0)
+			(effects
+				(font
+					(size 1.27 1.27)
+				)
+				(hide yes)
+			)
+		)
 		(pin "2"
 		)
@@
 			)
 		)
-		(property "LCSC Part #" "C19734"
+		(property "LCSC Part #" "C167747 "
 			(at 43.18 247.65 0)
 			(effects
@@
 			)
 		)
+		(property "LCSC Part #" "C2681320"
+			(at 157.48 267.97 0)
+			(effects
+				(font
+					(size 1.27 1.27)
+				)
+				(hide yes)
+			)
+		)
 		(pin "3"
 		)
@@
 			)
 		)
-		(property "LCSC Part #" "C2913202"
+		(property "LCSC Part #" "C2913205"
 			(at 104.14 49.53 0)
 			(effects
