File: Docs/Documents & Advanced/PCB/V3.3/einkPDA_keyboard/einkPDA_keyboard.kicad_sch (KiCad schematic)
At the start: 140 parts, among them J1 USB_C_Receptacle_USB2.0_16P, J2 Conn_01x12_Pin, J3 Conn_01x26_Pin, J4 Micro_SD_Card, J5 Conn_01x12_Pin, Q1 MMBT3904, SW36 YTS-C017-2B, SW4 SW_DIP_x02, SW41 YTS-C017-2B, U1 ESP32-S3-WROOM-1-N16R2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

Commit message: Update wiring for load switch
Parts:
- removed JP4, JP5: SolderJumper_3_Bridged12, Jumper:SolderJumper-3_P1.3mm_Bridged12_RoundedPad1.0x1.5mm, symbol Jumper:SolderJumper_3_Bridged12
- added R21, R22: 10k, Resistor_SMD:R_0805_2012Metric, symbol Device:R
Connections:
- net +3.3V: no longer R10.2, R9.1, RN3.1 (R1.1), RN3.2 (R2.1), RN3.3 (R3.1), RN3.4 (R4.1)
- net GND: now also C22.2; no longer C22.1
- net I2C_SCL: no longer J2.3 (Pin_3), J5.3 (Pin_3)
- net I2C_SDA: no longer J2.2 (Pin_2), J5.2 (Pin_2)
- net RX: now also J5.11 (Pin_11)
- net TX: now also J5.10 (Pin_10)
- net V_LOADSWITCH: now also C22.1, R10.2, R9.1, RN3.1 (R1.1), RN3.2 (R2.1), RN3.3 (R3.1), RN3.4 (R4.1), R21.2, R22.1; no longer C22.2
- net CHRG renamed I2C_SCL_SWITCHED
- net I2C_SCL_SWITCHED: now also J2.3 (Pin_3), J5.3 (Pin_3), R22.2
- net EX_D renamed I2C_SDA_SWITCHED
- net I2C_SDA_SWITCHED: now also J2.2 (Pin_2), J5.2 (Pin_2), R21.1
- net EX_E: no longer names the net of U1.25 (IO48)
- no-connect marks 9 -> 10
Other:
- moved on the sheet: C1, C22, R1, RN3, SW1, SW10, SW11, SW12, SW13, SW14, SW15, SW16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
