File: Resources/PCB/V3.5/einkPDA_screen/einkPDA_screen.kicad_pcb (KiCad board)
At the start: 2 copper layers, 95 x 54 mm, 28 parts, among them J3 CapacitiveTouch, J4 Conn_01x12_Pin, Q1 Si1308EDL, U1 MPR121QR2

Commit message: Update versioning
Other:
- board text added: "@Ashtf // V3.5"
- board text removed: "@Ashtf // V3.4"
